Commit message: update model and moveit_config

File: seed_r7_description/arm_typeA/arm.urdf (robot description, URDF)
Before this commit: robot SEED-Arm-Mover-typeA, 32 links, 31 joints
Links:
- link elbow_link: geometry collision cylinder length=0.15 radius=0.035; visual mesh filename=package://seed_r7_description/meshes/typeA_arm/elbow.dae scale=1 1 1
- link forearm_link: geometry collision box size=0.05 0.08 0.12; visual mesh filename=package://seed_r7_description/meshes/typeA_arm/forearm.dae scale=1 1 1
- link shoulder_link: geometry collision box size=0.07 0.05 0.05; visual mesh filename=package://seed_r7_description/meshes/typeA_arm/shoulder_p.d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 scale=1 1 1
- link upperarm_link: geometry collision box size=0.1 0.08 0.3; visual mesh filename=package://seed_r7_description/meshes/typeA_arm/upperarm.dae scale=1 1 1
Joints:
- joint wrist_r_joint: limit lower=-0.17 upper=0.17 effort=100 velocity=1.05 -> lower=-0.35 upper=0.35 effort=100 velocity=1.05

File: seed_r7_description/urdf/typeA_arm/arm_typea.urdf.xacro (robot description, xacro)
@@ -15,5 +15,5 @@
       <origin xyz="0 0 0.045" rpy="0 0 0"/>
       <geometry>
-        <cylinder length="0.07" radius="0.04"/>-->
+        <cylinder length="0.07" radius="0.04"/>
         <!--<mesh filename="package://seed_r7_description/meshes/typeA_arm/shoulder_y.dae" scale="1 1 1" />-->
       </geometry>
@@ -34,7 +34,8 @@
     </visual> </xacro:unless>
     <xacro:unless value="${disable_mesh}"> <collision>
-      <origin xyz="0 0 0.005" rpy="0 0 0"/>
-      <geometry>
-        <cylinder length="0.01" radius="0.04"/>-->
+      <origin xyz="-0.01 0 0.025" rpy="0 0 0"/>
+      <geometry>
+        <box size="0.07 0.05 0.05"/>
+        <!--<cylinder length="0.03" radius="0.04"/>-->
         <!--<mesh filename="package://seed_r7_description/meshes/typeA_arm/shoulder_p.dae" scale="1 1 1" />-->
       </geometry>
@@ -55,7 +56,8 @@
     </visual> </xacro:unless>
     <xacro:unless value="${disable_mesh}"> <collision>
-      <origin xyz="0 0 0.14" rpy="0 0 0"/>
-      <geometry>
-        <cylinder length="0.3" radius="0.04"/>-->
+      <origin xyz="-0.02 0 0.16" rpy="0 0 0"/>
+      <geometry>
+        <box size="0.1 0.08 0.3"/>
+        <!--<cylinder length="0.3" radius="0.04"/>-->
         <!--<mesh filename="package://seed_r7_description/meshes/typeA_arm/upperarm.dae" scale="1 1 1" />-->
       </geometry>
@@ -76,7 +78,7 @@
     </visual> </xacro:unless>
     <xacro:unless value="${disable_mesh}"> <collision>
-      <origin xyz="-0.022 0 0.05" rpy="0 0 0"/>
-      <geometry>
-        <cylinder length="0.15" radius="0.04"/>-->
+      <origin xyz="-0.03 0 0.06" rpy="0 0 0"/>
+      <geometry>
+        <cylinder length="0.15" radius="0.035"/>
         <!--<mesh filename="package://seed_r7_description/meshes/typeA_arm/elbow.dae" scale="1 1 1" />-->
       </geometry>
@@ -99,5 +101,6 @@
       <origin xyz="0 0 0.06" rpy="0 0 0"/>
       <geometry>
-        <cylinder length="0.12" radius="0.04"/>-->
+        <box size="0.05 0.08 0.12"/>
+        <!--<cylinder length="0.12" radius="0.04"/>-->
         <!--<mesh filename="package://seed_r7_description/meshes/typeA_arm/forearm.dae" scale="1 1 1" />-->
       </geometry>
@@ -120,5 +123,5 @@
       <origin xyz="0 0 0" rpy="1.57 1.57 0"/>
       <geometry>
-        <cylinder length="0.03" radius="0.005"/>-->
+        <cylinder length="0.03" radius="0.005"/>
         <!--<mesh filename="package://seed_r7_description/meshes/typeA_arm/wrist_r.dae" scale="1 1 1" />-->
       </geometry>
@@ -141,5 +144,5 @@
       <origin xyz="0 0 0" rpy="1.570 0 0"/>
       <geometry>
-        <cylinder length="0.03" radius="0.005"/>-->
+        <cylinder length="0.03" radius="0.005"/>
         <!--<mesh filename="package://seed_r7_description/meshes/typeA_arm/wrist_p.dae" scale="1 1 1" />-->
       </geometry>
@@ -197,5 +200,5 @@
     <axis   xyz="0 1 0"/>
     <!-- from -25 to 85 degrees-->
-    <limit lower="-0.17" upper="0.17" effort="100" velocity="1.05" />
+    <limit lower="-0.35" upper="0.35" effort="100" velocity="1.05" />
     <dynamics damping="0.2" friction="0" />
   </joint>
