Commit message: add camera link and modify gain

File: seed_r7_description/typef/noid.urdf.xacro (robot description, xacro)
@@ -11,4 +11,5 @@
  <!-- gazebo settings -->
  <!-- camera -->
+ <!--
  <link name="camera_frame" />
  <link name="camera_optical_frame" />
@@ -23,6 +24,39 @@
    <origin xyz="0 0 0" rpy="-1.570796326795 0 -1.570796326795" />
  </joint>
+ -->
+<!--
  <xacro:gazebo_camera link_name="camera_frame"
                       frame_name="camera_optical_frame" />
+-->
+<xacro:property  name="camera_name" value="front_camera"/>
+<link name="${camera_name}_depth_optical_frame"/>
+<joint name="${camera_name}_depth_optical_joint" type="fixed">
+  <origin xyz="0 0 0" rpy="${-M_PI/2} 0 ${-M_PI/2}" />
+  <parent link="${camera_name}_link" />
+  <child link="${camera_name}_depth_optical_frame" />
+</joint>
+<xacro:gazebo_depth_camera link_name="${camera_name}_link"
+                      frame_name="${camera_name}_depth_optical_frame"
+                      camera_name="${camera_name}"/>/>
+<xacro:property  name="camera_name" value="rear_camera"/>
+<link name="${camera_name}_depth_optical_frame"/>
+<joint name="${camera_name}_depth_optical_joint" type="fixed">
+  <origin xyz="0 0 0" rpy="${-M_PI/2} 0 ${-M_PI/2}" />
+  <parent link="${camera_name}_link" />
+  <child link="${camera_name}_depth_optical_frame" />
+</joint>
+<xacro:gazebo_depth_camera link_name="${camera_name}_link"
+                      frame_name="${camera_name}_depth_optical_frame"
+                      camera_name="${camera_name}"/>/>
+<xacro:property  name="camera_name" value="chest_camera"/>
+<link name="${camera_name}_depth_optical_frame"/>
+<joint name="${camera_name}_depth_optical_joint" type="fixed">
+  <origin xyz="0 0 0" rpy="${-M_PI/2} 0 ${-M_PI/2}" />
+  <parent link="${camera_name}_link" />
+  <child link="${camera_name}_depth_optical_frame" />
+</joint>
+<xacro:gazebo_depth_camera link_name="${camera_name}_link"
+                      frame_name="${camera_name}_depth_optical_frame"
+                      camera_name="${camera_name}"/>/>
  <!-- laser -->
  <xacro:gazebo_laser_sensor link_name="wheels_base_laser_link"
@@ -37,13 +71,13 @@
      <!-- lifter -->
      <mimic joint="knee_joint"  offset="0.0" multiplier="-1.0"
-            P="4000" I="0.1" D="80" i_max="500" i_min="-500"
-            command_max="2000" command_min="-2000">
+            P="100" I="0.1" D="10" i_max="500" i_min="-500"
+            command_max="2000" command_min="-2000" velocity='true'>
        knee_joint_mimic
        <joint> knee_joint </joint>
        <offset> 0.0 </offset>
        <multiplier> -1.0 </multiplier>
-       <P> 4000 </P>
+       <P> 100 </P>
        <I> 0.1 </I>
-       <D> 80 </D>
+       <D> 10 </D>
        <i_max>  500 </i_max>
        <i_min> -500 </i_min>
@@ -52,13 +86,13 @@
      </mimic>
      <mimic joint="ankle_joint"  offset="0.0" multiplier="-1.0"
-            P="4000" I="0.1" D="80" i_max="500" i_min="-500"
-            command_max="2000" command_min="-2000">
+            P="100" I="0.1" D="10" i_max="500" i_min="-500"
+            command_max="2000" command_min="-2000" velocity='true'>
        ankle_joint_mimic
        <joint> ankle_joint </joint>
        <offset> 0.0 </offset>
        <multiplier> -1.0 </multiplier>
-       <P> 4000 </P>
+       <P> 100 </P>
        <I> 0.1 </I>
-       <D> 80 </D>
+       <D> 10 </D>
        <i_max>  500 </i_max>
        <i_min> -500 </i_min>
@@ -68,13 +102,13 @@
      <!-- lifter(dummy) -->
      <mimic joint="knee_joint"  offset="0.0" multiplier="-1.0"
-            P="1000" I="0.0" D="1" i_max="0" i_min="0"
-            command_max="200" command_min="-200">
+            P="100" I="0.0" D="10" i_max="0" i_min="0"
+            command_max="200" command_min="-200" velocity='true'>
        knee_joint_dummy
        <joint> knee_joint </joint>
        <offset> 0.0 </offset>
        <multiplier> -1.0 </multiplier>
-       <P> 1000 </P>
-       <I> 0.0 </I>
-       <D> 1 </D>
+       <P> 100 </P>
+       <I> 0.0 </I>
+       <D> 10 </D>
        <i_max>  0 </i_max>
        <i_min> -0 </i_min>
@@ -83,13 +117,13 @@
      </mimic>
      <mimic joint="ankle_joint"  offset="0.0" multiplier="1.0"
-            P="1000" I="0.0" D="1" i_max="0" i_min="0"
-            command_max="200" command_min="-200">
+            P="100" I="0.0" D="10" i_max="0" i_min="0"
+            command_max="200" command_min="-200"  velocity='true'>
        ankle_joint_dummy
        <joint> ankle_joint </joint>
        <offset> 0.0 </offset>
        <multiplier> 1.0 </multiplier>
-       <P> 1000 </P>
-       <I> 0.0 </I>
-       <D> 1 </D>
+       <P> 100 </P>
+       <I> 0.0 </I>
+       <D> 10 </D>
        <i_max>  0 </i_max>
        <i_min> -0 </i_min>

File: seed_r7_description/urdf/typeF_upperbody/noid_upper_typef.urdf.xacro (robot description, xacro)
@@ -576,4 +576,16 @@
   </joint>
   <xacro:gazebo_transmission joint_name="r_wrist_r_joint" />
+  <link name="chest_camera_link"/>
+    <joint name="body_link_to_chest_camera_link" type="fixed">
+      <parent  link="body_link"/>
+      <child link="chest_camera_link"/>
+      <origin xyz="0.062143 0.0 0.322289 " rpy="0 0.785398 0"/>
+    </joint>
+    <link name="chest_camera_right_ir_frame"/>
+    <joint name="chest_camera_link_to_chest_camera_right_ir_link" type="fixed">
+      <parent  link="chest_camera_link"/>
+      <child link="chest_camera_right_ir_frame"/>
+      <origin xyz="0 -0.055 0" rpy="0 0 0"/>  <!-- realsense d415-->
+    </joint>
   </xacro:macro>
 </robot>
